File: SD_IDE_IPOD.kicad_sch (KiCad schematic)
At the start: 18 parts, among them P1 FPCConnector 40PIN 0.5MM, U1 FC1307A, U2 P25Q20H-SSH-IT

Commit message: Wired Most connections
Parts:
- added R11, R13, R14: 100m, easyeda2kicad:R0402, symbol easyeda2kicad:RTT02R100FTH
- added R12: 10k, easyeda2kicad:R0402, symbol easyeda2kicad:0402WGJ0103TCE
Connections:
- net APQ is gone; now on net DMARQ: P1.19
- net DASP is gone; now on net nDASP: P1.4, U1.60 (nDASP)
- net HA9 is gone; now on net nIOR: P1.16
- net +3.3V: no longer P1.2, P1.3
- net CE1: now also U1.95 (CE2), U1.96 (CE1)
- net GND: now also U1.1 (GND), U1.105 (IO_GND), U1.11 (GND), U1.118 (CORE_GND), U1.23 (CORE_GND), U1.26 (AS18), U1.28 (DVSS_LVD), U1.30 (VSS_LVD), U1.32 (VSS_LDO), U1.34 (AGND_PLL), U1.36 (DGND_PLL), U1.38 (F_VSS), U1.46 (GND), U1.51 (nIOIS16), U1.55 (IO_GND), U1.65 (CORE_GND), U1.72 (HA4), U1.73 (HA5), U1.74 (nCSEL), U1.76 (CORE_GND), U1.78 (HA6), U1.80 (HA7), U1.87 (CORE_GND), U1.89 (HA8), U1.91 (HA9), U1.93 (HOE), U1.94 (HA10), U1.98 (GND), R11.2, R12.1, R13.2, R14.2
- net HA2: now also U1.68 (HA2)
- net HD11: now also U1.109 (HD11)
- net HD12: now also U1.107 (HD12)
- net HD13: now also U1.103 (HD13)
- net HD14: now also U1.101 (HD14)
- net HD15: now also U1.99 (HD15)
- net HD4: now also U1.108 (HD4)
- net HD5: now also U1.104 (HD5)
- net HD6: now also U1.102 (HD6)
- net HD7: now also U1.100 (HD7)
- net INTRQ: now also U1.71 (nRST), U1.79 (INTRQ)
- net nIOR: now also U1.92 (nIOR); no longer P1.17
- net VCC3.3: now reaches U1.10 (IO_PWR_33)
- net VCC3.3: now also P1.2, P1.3, U1.106 (IO_PWR_33), U1.117 (IO_PWR_33), U1.128 (IO_PWR_33), U1.19 (IO_PWR_33), U1.31 (DVDD_LVD), U1.33 (DVDD_LDO), U1.44 (IO_PWR_33), U1.54 (IO_PWR_33), U1.66 (IO_PWR_33), U1.77 (IO_PWR_33), U1.81 (WE), U1.88 (IO_PWR_33), U1.97 (IO_PWR_33)
- net HD3: now reaches U1.110 (HD3)
- net VCC1.8: now reaches U1.119 (CORE_PWR_18)
- net VCC1.8: now also U1.12 (CORE_PWR_18), U1.24 (CORE_PWR_18), U1.25 (VDD_LVD), U1.27 (AV18), U1.29 (VDD_18V), U1.35 (AVDD_PLL), U1.37 (DVDD_PLL), U1.39 (F_VPP), U1.40 (F_VDD), U1.45 (CORE_PWR_18), U1.64 (CORE_PWR_18), U1.75 (CORE_PWR_18), U1.86 (CORE_PWR_18)
- net at U1.14 (IOP2): now also R14.1
- net nDASP: now reaches U1.50 (HD10)
- net nDASP: now also U1.52 (HD9), U1.53 (HD2), U1.56 (HD8), U1.57 (HD1), U1.58 (STSCHG), U1.59 (HD0), U1.61 (HA0), U1.62 (REG), U1.63 (HA1)
- net DMARQ: now reaches U1.67 (DMARQ)
- net IORDY: now reaches U1.69 (IORDY)
- net at U1.7 (IOP4): now also R11.1
- net at U1.8 (IOP5): now also R13.1
- net at U1.85 (IOP6): now also R12.2
- net nIOW: now reaches U1.90 (nIOW)
- net nIOW: now also P1.17
- net HA3 renamed I0RDY
- no-connect marks 3 -> 25
Other:
- moved on the sheet: U1

Commit message: dev: added LDO and ERC rules
Parts:
- added C14, C16: 1uF, symbol Device:C
- added C15, C17: 0.1uF, symbol Device:C
- added R15, R16: 10k, symbol Device:R
- added U7: AMS1117-1.8, symbol Regulator_Linear:AMS1117CD-1.8
Connections:
- net CD is gone; now on net +1V8: Card1.9 (CD), Card2.9 (CD)
- net CE2 is gone; now on net CE1: P1.5
- net GND is gone; now on net +1V8: C1.2, C2.2, C3.2, Card1.10 (G3), Card1.11 (G4), Card1.12 (G1), Card1.13 (G2), Card1.6 (VSS), Card2.10 (G3), Card2.11 (G4), Card2.12 (G1), Card2.13 (G2), Card2.6 (VSS), P1.13, P1.15, P1.18, P1.20, P1.37, P1.41, P1.42, R11.2, R12.1, R13.2, R14.2, U1.1 (GND), U1.105 (IO_GND), U1.11 (GND), U1.118 (CORE_GND), U1.23 (CORE_GND), U1.26 (AS18), U1.28 (DVSS_LVD), U1.30 (VSS_LVD), U1.32 (VSS_LDO), U1.34 (AGND_PLL), U1.36 (DGND_PLL), U1.38 (F_VSS), U1.46 (GND), U1.51 (nIOIS16), U1.55 (IO_GND), U1.65 (CORE_GND), U1.72 (HA4), U1.73 (HA5), U1.74 (nCSEL), U1.76 (CORE_GND), U1.78 (HA6), U1.80 (HA7), U1.87 (CORE_GND), U1.89 (HA8), U1.91 (HA9), U1.93 (HOE), U1.94 (HA10), U1.98 (GND), U2.4 (GND)
- net HA1 is gone; now on net HA0: P1.10
- net HD0 is gone; now on net HA0: P1.22
- net HD1 is gone; now on net HA0: P1.24
- net HD10 is gone; now on net HA0: P1.31
- net HD2 is gone; now on net HA0: P1.26
- net HD8 is gone; now on net HA0: P1.35
- net HD9 is gone; now on net HA0: P1.33
- net REG is gone; now on net HA0: P1.12
- net SD0_CMD is gone; now on net SD0_CLK: Card1.3 (CMD), R3.2, U1.115 (SD0_CLK)
- net SD0_DAT1 is gone; now on net SD0_CLK: Card1.8 (DAT1), R5.2, U1.113 (SD0_DAT1), U1.116 (SD0_CMD)
- net SD1_DAT2 is gone; now on net SD1_DAT1: Card2.1 (DAT2), R6.2, U1.126 (SD1_DAT3)
- net SD1_DAT3 is gone; now on net SD1_DAT1: Card2.2 (CD/DAT3), R7.2
- net STSCHG is gone; now on net HA0: P1.9
- net VCC1.8 is gone; now on net +1V8: U1.119 (CORE_PWR_18), U1.12 (CORE_PWR_18), U1.24 (CORE_PWR_18), U1.25 (VDD_LVD), U1.27 (AV18), U1.29 (VDD_18V), U1.35 (AVDD_PLL), U1.37 (DVDD_PLL), U1.39 (F_VPP), U1.40 (F_VDD), U1.45 (CORE_PWR_18), U1.64 (CORE_PWR_18), U1.75 (CORE_PWR_18), U1.86 (CORE_PWR_18)
- net VCC3.3 is gone; now on net +1V8: P1.2, P1.3, U1.10 (IO_PWR_33), U1.106 (IO_PWR_33), U1.117 (IO_PWR_33), U1.128 (IO_PWR_33), U1.19 (IO_PWR_33), U1.31 (DVDD_LVD), U1.33 (DVDD_LDO), U1.44 (IO_PWR_33), U1.54 (IO_PWR_33), U1.66 (IO_PWR_33), U1.77 (IO_PWR_33), U1.81 (WE), U1.88 (IO_PWR_33), U1.97 (IO_PWR_33)
- net nDASP is gone; now on net HA0: P1.4, U1.50 (HD10), U1.52 (HD9), U1.53 (HD2), U1.56 (HD8), U1.57 (HD1), U1.58 (STSCHG), U1.59 (HD0), U1.60 (nDASP), U1.61 (HA0), U1.62 (REG), U1.63 (HA1)
- net nRST is gone; now on net INTRQ: P1.38
- net SD1_DAT1: now also R16.2
- net HA3: now reaches U1.70 (HA3)
- net ICLKSEL: now reaches U1.82 (ICLKSEL)
- net +3.3V renamed +1V8
- net +1V8: now also C14.1, C14.2, C15.1, C15.2, C16.1, C16.2, C17.1, C17.2, R15.1, R15.2, R16.1
